Commit message: Add simulated camera with image stream
- Add URDF macros for cameras
- Add Gazebo plugin for image stream
- Add ros_gz_bridge params

File: ur_handeye_description/urdf/ur_handeye_workcell.urdf.xacro (robot description, xacro)
@@ -22,3 +22,35 @@
       <origin xyz="0 0 1" rpy="0 0 0" />
   </xacro:ur_handeye_workcell>
+  <!-- Check eye-in-hand configuration -->
+  <joint name="robot_to_camera_in_hand" type="fixed">
+    <parent link="tool0"/>
+    <child link="camera_in_hand_base_link"/>
+    <origin xyz="0 0 0" rpy="0 0 ${pi}" />
+  </joint>
+  <link name="camera_in_hand_base_link" />
+  <xacro:sensor_d435
+    parent="camera_in_hand_base_link"
+    name="camera_in_hand"
+    use_nominal_extrinsics="true"
+    add_plug="false"
+    use_mesh="true"
+  >
+    <origin xyz="0 0 0" rpy="0 0 0"/>
+  </xacro:sensor_d435>
+  <!-- Check eye-to-hand configuration -->
+  <joint name="robot_to_camera_to_hand" type="fixed">
+    <parent link="world"/>
+    <child link="camera_to_hand_base_link"/>
+    <origin xyz="0 0.5 2" rpy="0 ${pi/6} 0 " />
+  </joint>
+  <link name="camera_to_hand_base_link" />
+  <xacro:sensor_d435
+    parent="camera_to_hand_base_link"
+    name="camera_to_hand"
+    use_nominal_extrinsics="true"
+    add_plug="false"
+    use_mesh="true"
+  >
+    <origin xyz="0 0 0" rpy="0 0 0"/>
+  </xacro:sensor_d435>
 </robot>

File: ur_handeye_description/urdf/ur_handeye_workcell_macro.xacro (robot description, xacro)
@@ -2,4 +2,5 @@
 <robot xmlns:xacro="http://ros.org/wiki/xacro">
   <xacro:include filename="$(find ur_description)/urdf/ur_macro.xacro"/>
+  <xacro:include filename="$(find ur_handeye_description)/urdf/cameras/_d435.urdf.xacro"/>
   <xacro:macro name="ur_handeye_workcell" params="
     name

File: ur_handeye_simulation/urdf/ur_handeye_workcell.urdf.xacro (robot description, xacro)
@@ -2,4 +2,5 @@
 <robot name="ur_handeye_workcell" xmlns:xacro="http://ros.org/wiki/xacro">
   <xacro:include filename="$(find ur_handeye_description)/urdf/ur_handeye_workcell_macro.xacro"/>
+  <xacro:include filename="$(find ur_handeye_simulation)/urdf/ur_handeye_camera_macro.xacro"/>
   <xacro:include filename="$(find ur_simulation_gz)/urdf/ur_gz.ros2_control.xacro" />
   <xacro:arg name="ur_type" default="ur20"/>
@@ -32,4 +33,11 @@
       <origin xyz="0 0 1" rpy="0 0 0" />
   </xacro:ur_handeye_workcell>
+  <!-- HAND-EYE-->
+  <xacro:handeye_camera
+    name="eye_to_hand_camera"
+    parent="world"
+  >
+    <origin xyz="0 0.5 2" rpy="0 ${pi/6} 0 " />
+  </xacro:handeye_camera>
   <!-- GAZEBO -->
   <gazebo>

Commit message: Minor adjustment in workcell description

File: ur_handeye_description/urdf/ur_handeye_workcell.urdf.xacro (robot description, xacro)
@@ -2,5 +2,5 @@
 <robot name="ur_handeye_workcell" xmlns:xacro="http://ros.org/wiki/xacro">
   <xacro:include filename="$(find ur_handeye_description)/urdf/ur_handeye_workcell_macro.xacro"/>
-  <xacro:arg name="ur_type" default="ur20"/>
+  <xacro:arg name="ur_type" default="ur10"/>
   <xacro:arg name="name" default="ur"/>
   <xacro:arg name="tf_prefix" default="" />
@@ -22,35 +22,3 @@
       <origin xyz="0 0 1" rpy="0 0 0" />
   </xacro:ur_handeye_workcell>
-  <!-- Check eye-in-hand configuration -->
-  <joint name="robot_to_camera_in_hand" type="fixed">
-    <parent link="tool0"/>
-    <child link="camera_in_hand_base_link"/>
-    <origin xyz="0 0 0" rpy="0 0 ${pi}" />
-  </joint>
-  <link name="camera_in_hand_base_link" />
-  <xacro:sensor_d435
-    parent="camera_in_hand_base_link"
-    name="camera_in_hand"
-    use_nominal_extrinsics="true"
-    add_plug="false"
-    use_mesh="true"
-  >
-    <origin xyz="0 0 0" rpy="0 0 0"/>
-  </xacro:sensor_d435>
-  <!-- Check eye-to-hand configuration -->
-  <joint name="robot_to_camera_to_hand" type="fixed">
-    <parent link="world"/>
-    <child link="camera_to_hand_base_link"/>
-    <origin xyz="0 0.5 2" rpy="0 ${pi/6} 0 " />
-  </joint>
-  <link name="camera_to_hand_base_link" />
-  <xacro:sensor_d435
-    parent="camera_to_hand_base_link"
-    name="camera_to_hand"
-    use_nominal_extrinsics="true"
-    add_plug="false"
-    use_mesh="true"
-  >
-    <origin xyz="0 0 0" rpy="0 0 0"/>
-  </xacro:sensor_d435>
 </robot>
