Commit message: Add Gazebo simulation for the robot workcell

File: ur_handeye_description/urdf/ur_handeye_workcell_macro.xacro (robot description, xacro)
@@ -3,11 +3,16 @@
   <xacro:include filename="$(find ur_description)/urdf/ur_macro.xacro"/>
   <xacro:macro name="ur_handeye_workcell" params="
+    name
+    tf_prefix
     parent
     *origin
-    ur_type
     joint_limits_parameters_file
     kinematics_parameters_file
     physical_parameters_file
     visual_parameters_file
+    safety_limits:=false
+    safety_pos_margin:=0.15
+    safety_k_position:=20
+    force_abs_paths:=false
     ">
     <material name="white">
@@ -18,5 +23,6 @@
       <visual>
         <geometry>
-          <mesh filename="package://ur_handeye_description/meshes/fzi_table.dae"/>
+          <box size="1.50 1.00 2"/>
+          <!-- <mesh filename="package://ur_handeye_description/meshes/fzi_table.dae"/> -->
         </geometry>
         <origin rpy="0 0 0" xyz="0.75 0.5 -1"/>
@@ -24,5 +30,6 @@
       <collision>
         <geometry>
-          <mesh filename="package://ur_handeye_description/meshes/fzi_table.dae"/>
+          <box size="1.50 1.00 2"/>
+          <!-- <mesh filename="package://ur_handeye_description/meshes/fzi_table.dae"/> -->
         </geometry>
         <origin rpy="0 0 0" xyz="0.75 0.5 -1"/>
@@ -37,5 +44,6 @@
       <visual>
         <geometry>
-          <mesh filename="package://ur_handeye_description/meshes/fzi_table.dae"/>
+          <box size="1.50 1.00 2"/>
+          <!-- <mesh filename="package://ur_handeye_description/meshes/fzi_table.dae"/> -->
         </geometry>
         <origin rpy="0 0 0" xyz="0.75 0.5 -1"/>
@@ -43,5 +51,6 @@
       <collision>
         <geometry>
-          <mesh filename="package://ur_handeye_description/meshes/fzi_table.dae"/>
+          <box size="1.50 1.00 2"/>
+          <!-- <mesh filename="package://ur_handeye_description/meshes/fzi_table.dae"/> -->
         </geometry>
         <origin rpy="0 0 0" xyz="0.75 0.5 -1"/>
@@ -56,10 +65,12 @@
       <visual>
         <geometry>
-          <mesh filename="package://ur_handeye_description/meshes/171005_Motek_Monitor_L.dae"/>
+          <box size="0.5 0.1 0.5"/>
+          <!-- <mesh filename="package://ur_handeye_description/meshes/171005_Motek_Monitor_L.dae"/> -->
         </geometry>
       </visual>
       <collision>
         <geometry>
-          <mesh filename="package://ur_handeye_description/meshes/171005_Motek_Monitor_L.dae"/>
+          <box size="0.5 0.1 0.5"/>
+          <!-- <mesh filename="package://ur_handeye_description/meshes/171005_Motek_Monitor_L.dae"/> -->
         </geometry>
       </collision>
@@ -78,6 +89,6 @@
     <!--This will create the specific robot-->
     <xacro:ur_robot
-      name="${ur_type}"
-      tf_prefix="${ur_type}_"
+      name="${name}"
+      tf_prefix="${tf_prefix}"
       parent="robot_mount"
       joint_limits_parameters_file="${joint_limits_parameters_file}"
@@ -85,4 +96,8 @@
       physical_parameters_file="${physical_parameters_file}"
       visual_parameters_file="${visual_parameters_file}"
+      safety_limits="${safety_limits}"
+      safety_pos_margin="${safety_pos_margin}"
+      safety_k_position="${safety_k_position}"
+      force_abs_paths="true"
     >
       <origin xyz="0 0 0" rpy="0 0 0" />

File: ur_handeye_simulation/urdf/ur_handeye_workcell.urdf.xacro (robot description, xacro)
@@ -2,4 +2,5 @@
 <robot name="ur_handeye_workcell" xmlns:xacro="http://ros.org/wiki/xacro">
   <xacro:include filename="$(find ur_handeye_description)/urdf/ur_handeye_workcell_macro.xacro"/>
+  <xacro:include filename="$(find ur_simulation_gz)/urdf/ur_gz.ros2_control.xacro" />
   <xacro:arg name="ur_type" default="ur20"/>
   <xacro:arg name="name" default="ur"/>
@@ -9,4 +10,10 @@
   <xacro:arg name="physical_parameters_file" default="$(find ur_description)/config/$(arg ur_type)/physical_parameters.yaml"/>
   <xacro:arg name="visual_parameters_file" default="$(find ur_description)/config/$(arg ur_type)/visual_parameters.yaml"/>
+  <xacro:arg name="safety_limits" default="false"/>
+  <xacro:arg name="safety_pos_margin" default="0.15"/>
+  <xacro:arg name="safety_k_position" default="20"/>
+  <xacro:arg name="simulation_controllers" default="$(find ur_simulation_gz)/config/ur_controllers.yaml" />
+  <xacro:arg name="transmission_hw_interface" default=""/>
+  <xacro:arg name="ros_namespace" default="" />
   <link name="world"/>
   <!--This will create the scene where the robot is located in-->
@@ -19,6 +26,25 @@
     physical_parameters_file="$(arg physical_parameters_file)"
     visual_parameters_file="$(arg visual_parameters_file)"
+    safety_limits="$(arg safety_limits)"
+    safety_pos_margin="$(arg safety_pos_margin)"
+    safety_k_position="$(arg safety_k_position)"
     >
       <origin xyz="0 0 1" rpy="0 0 0" />
   </xacro:ur_handeye_workcell>
+  <!-- GAZEBO -->
+  <gazebo>
+    <plugin name="gz::sim::systems::Sensors" filename="gz-sim-sensors-system"/>
+    <plugin filename="gz_ros2_control-system" name="gz_ros2_control::GazeboSimROS2ControlPlugin">
+      <parameters>$(arg simulation_controllers)</parameters>
+      <ros>
+        <namespace>$(arg ros_namespace)</namespace>
+      </ros>
+    </plugin>
+  </gazebo>
+  <!-- ros2 control instance -->
+  <xacro:ur_ros2_control
+    name="$(arg name)"
+    tf_prefix="$(arg tf_prefix)"
+    transmission_hw_interface="$(arg transmission_hw_interface)"
+  />
 </robot>

Commit message: Fix Gazebo mesh visualization
Set GZ_SIM_RESOURCE_PATH in launch file pointing to "<pkg_name>/share"

File: ur_handeye_description/urdf/ur_handeye_workcell_macro.xacro (robot description, xacro)
@@ -23,6 +23,5 @@
       <visual>
         <geometry>
-          <box size="1.50 1.00 2"/>
-          <!-- <mesh filename="package://ur_handeye_description/meshes/fzi_table.dae"/> -->
+          <mesh filename="package://ur_handeye_description/meshes/fzi_table.dae"/>
         </geometry>
         <origin rpy="0 0 0" xyz="0.75 0.5 -1"/>
@@ -30,9 +29,14 @@
       <collision>
         <geometry>
-          <box size="1.50 1.00 2"/>
-          <!-- <mesh filename="package://ur_handeye_description/meshes/fzi_table.dae"/> -->
+          <mesh filename="package://ur_handeye_description/meshes/fzi_table.dae"/>
         </geometry>
         <origin rpy="0 0 0" xyz="0.75 0.5 -1"/>
       </collision>
+      <inertial>
+    <mass value="2"/>
+    <inertia ixx="0.0001" ixy="0" ixz="0"
+              iyy="0.0001" iyz="0"
+              izz="0.0001"/>
+  </inertial>
     </link>
     <joint name="ground_to_table1" type="fixed">
@@ -44,6 +48,5 @@
       <visual>
         <geometry>
-          <box size="1.50 1.00 2"/>
-          <!-- <mesh filename="package://ur_handeye_description/meshes/fzi_table.dae"/> -->
+          <mesh filename="package://ur_handeye_description/meshes/fzi_table.dae"/>
         </geometry>
         <origin rpy="0 0 0" xyz="0.75 0.5 -1"/>
@@ -51,9 +54,14 @@
       <collision>
         <geometry>
-          <box size="1.50 1.00 2"/>
-          <!-- <mesh filename="package://ur_handeye_description/meshes/fzi_table.dae"/> -->
+          <mesh filename="package://ur_handeye_description/meshes/fzi_table.dae"/>
         </geometry>
         <origin rpy="0 0 0" xyz="0.75 0.5 -1"/>
       </collision>
+      <inertial>
+    <mass value="2"/>
+    <inertia ixx="0.0001" ixy="0" ixz="0"
+              iyy="0.0001" iyz="0"
+              izz="0.0001"/>
+  </inertial>
     </link>
     <joint name="ground_to_table2" type="fixed">
@@ -65,12 +73,10 @@
       <visual>
         <geometry>
-          <box size="0.5 0.1 0.5"/>
-          <!-- <mesh filename="package://ur_handeye_description/meshes/171005_Motek_Monitor_L.dae"/> -->
+          <mesh filename="package://ur_handeye_description/meshes/171005_Motek_Monitor_L.dae"/>
         </geometry>
       </visual>
       <collision>
         <geometry>
-          <box size="0.5 0.1 0.5"/>
-          <!-- <mesh filename="package://ur_handeye_description/meshes/171005_Motek_Monitor_L.dae"/> -->
+          <mesh filename="package://ur_handeye_description/meshes/171005_Motek_Monitor_L.dae"/>
         </geometry>
       </collision>

Commit message: Add MoveIt to control the simulated robot

File: ur_handeye_description/urdf/ur_handeye_workcell_macro.xacro (robot description, xacro)
@@ -92,5 +92,5 @@
       <parent link="table2"/>
       <child link="robot_mount"/>
-      <origin xyz="1.1 0.5 0" rpy="0 0 ${pi}" />
+      <origin xyz="1.0 0.5 0" rpy="0 0 ${pi}" />
     </joint>
     <!--This will create the specific robot-->

File: ur_handeye_simulation/urdf/ur_handeye_workcell.urdf.xacro (robot description, xacro)
@@ -4,5 +4,5 @@
   <xacro:include filename="$(find ur_handeye_simulation)/urdf/ur_handeye_camera_macro.xacro"/>
   <xacro:include filename="$(find ur_simulation_gz)/urdf/ur_gz.ros2_control.xacro" />
-  <xacro:arg name="ur_type" default="ur20"/>
+  <xacro:arg name="ur_type" default="ur10"/>
   <xacro:arg name="name" default="ur"/>
   <xacro:arg name="tf_prefix" default="" />
@@ -14,5 +14,5 @@
   <xacro:arg name="safety_pos_margin" default="0.15"/>
   <xacro:arg name="safety_k_position" default="20"/>
-  <xacro:arg name="simulation_controllers" default="$(find ur_simulation_gz)/config/ur_controllers.yaml" />
+  <xacro:arg name="simulation_controllers" default="$(find ur_handeye_simulation)/config/ur_controllers.yaml" />
   <xacro:arg name="transmission_hw_interface" default=""/>
   <xacro:arg name="ros_namespace" default="" />
