Commit message: Add option for pattern as URDF
- visualization works in both RViz and Gazebo

File: ur_handeye_simulation/urdf/ur_handeye_workcell.urdf.xacro (robot description, xacro)
@@ -3,4 +3,5 @@
   <xacro:include filename="$(find ur_handeye_description)/urdf/ur_handeye_workcell_macro.xacro"/>
   <xacro:include filename="$(find ur_handeye_simulation)/urdf/ur_handeye_camera_macro.xacro"/>
+  <xacro:include filename="$(find ur_handeye_simulation)/urdf/ur_handeye_pattern_macro.xacro"/>
   <xacro:include filename="$(find ur_simulation_gz)/urdf/ur_gz.ros2_control.xacro" />
   <xacro:arg name="ur_type" default="ur10"/>
@@ -40,4 +41,14 @@
     <origin xyz="0 0.5 2" rpy="0 ${pi/6} 0 " />
   </xacro:handeye_camera>
+  <!-- PATTERN -->
+  <xacro:handeye_pattern
+    name="pattern"
+    parent="world"
+    width="0.9"
+    height="0.8"
+    texture_path="$(find ur_handeye_simulation)/models/textures/pattern2.png"
+  >
+    <origin xyz="1.5 0.5 1.05" rpy="0 0 0 " />
+  </xacro:handeye_pattern>
   <!-- GAZEBO -->
   <gazebo>

Commit message: Generalize code to support both handeye setups

File: ur_handeye_simulation/urdf/ur_handeye_workcell.urdf.xacro (robot description, xacro)
@@ -5,4 +5,6 @@
   <xacro:include filename="$(find ur_handeye_simulation)/urdf/ur_handeye_pattern_macro.xacro"/>
   <xacro:include filename="$(find ur_simulation_gz)/urdf/ur_gz.ros2_control.xacro" />
+  <!-- options: eye_to_hand, eye_in_hand -->
+  <xacro:arg name="handeye_setup" default="eye_in_hand"/>
   <xacro:arg name="ur_type" default="ur10"/>
   <xacro:arg name="name" default="ur"/>
@@ -34,21 +36,44 @@
       <origin xyz="0 0 1" rpy="0 0 0" />
   </xacro:ur_handeye_workcell>
-  <!-- HAND-EYE-->
-  <xacro:handeye_camera
-    name="eye_to_hand_camera"
-    parent="world"
-  >
-    <origin xyz="0 0.5 2" rpy="0 ${pi/6} 0 " />
-  </xacro:handeye_camera>
-  <!-- PATTERN -->
-  <xacro:handeye_pattern
-    name="pattern"
-    parent="world"
-    width="0.9"
-    height="0.8"
-    texture_path="$(find ur_handeye_simulation)/models/textures/pattern2.png"
-  >
-    <origin xyz="1.5 0.5 1.05" rpy="0 0 0 " />
-  </xacro:handeye_pattern>
+  <!-- ============================================================================ -->
+  <!-- Hand-eye setups settings                                                     -->
+  <!-- ============================================================================ -->
+  <xacro:property name="setup" value="$(arg handeye_setup)"/>
+  <!-- Eye-to-Hand -->
+  <xacro:if value="${setup == 'eye_to_hand'}">
+    <xacro:handeye_camera
+      name="eye_to_hand_camera"
+      parent="world"
+    >
+      <origin xyz="0 0.5 2" rpy="0 ${pi/6} 0" />
+    </xacro:handeye_camera>
+    <xacro:handeye_pattern
+      name="pattern"
+      parent="tool0"
+      width="0.9"
+      height="0.8"
+      texture_path="$(find ur_handeye_simulation)/models/textures/pattern2.png"
+    >
+      <origin xyz="0 0 0.05" rpy="0 0 0" />
+    </xacro:handeye_pattern>
+  </xacro:if>
+  <xacro:if value="${setup == 'eye_in_hand'}">
+    <xacro:handeye_camera
+      name="eye_in_hand_camera"
+      parent="tool0"
+    >
+      <origin xyz="0 -0.05 0.02" rpy="${pi/2} ${-pi/2} 0" />
+    </xacro:handeye_camera>
+    <xacro:handeye_pattern
+      name="pattern"
+      parent="world"
+      width="0.9"
+      height="0.8"
+      texture_path="$(find ur_handeye_simulation)/models/textures/pattern2.png"
+    >
+      <origin xyz="1.5 0.5 1.05" rpy="0 0 0" />
+    </xacro:handeye_pattern>
+  </xacro:if>
+  <!-- ============================================================================ -->
   <!-- GAZEBO -->
   <gazebo>

Commit message: Update pattern textures

File: ur_handeye_simulation/urdf/ur_handeye_workcell.urdf.xacro (robot description, xacro)
@@ -40,4 +40,7 @@
   <!-- ============================================================================ -->
   <xacro:property name="setup" value="$(arg handeye_setup)"/>
+  <xacro:property name="pattern_width"   value="0.200"/>
+  <xacro:property name="pattern_height"  value="0.200"/>
+  <xacro:property name="pattern_texture" value="checker_200x200_8x9_20.png"/>
   <!-- Eye-to-Hand -->
   <xacro:if value="${setup == 'eye_to_hand'}">
@@ -51,7 +54,7 @@
       name="pattern"
       parent="tool0"
-      width="0.9"
-      height="0.8"
-      texture_path="$(find ur_handeye_simulation)/models/textures/pattern2.png"
+      width="${pattern_width}"
+      height="${pattern_height}"
+      texture_path="$(find ur_handeye_simulation)/models/textures/${pattern_texture}"
     >
       <origin xyz="0 0 0.05" rpy="0 0 0" />
@@ -68,7 +71,7 @@
       name="pattern"
       parent="world"
-      width="0.9"
-      height="0.8"
-      texture_path="$(find ur_handeye_simulation)/models/textures/pattern2.png"
+      width="${pattern_width}"
+      height="${pattern_height}"
+      texture_path="$(find ur_handeye_simulation)/models/textures/${pattern_texture}"
     >
       <origin xyz="1.5 0.5 1.05" rpy="0 0 0" />

Commit message: Test corner detection

File: ur_handeye_simulation/urdf/ur_handeye_workcell.urdf.xacro (robot description, xacro)
@@ -75,5 +75,5 @@
       texture_path="$(find ur_handeye_simulation)/models/textures/${pattern_texture}"
     >
-      <origin xyz="1.5 0.5 1.05" rpy="0 0 0" />
+      <origin xyz="1.8 0.4 1.05" rpy="0 0 0" />
     </xacro:handeye_pattern>
   </xacro:if>

Commit message: Add spawner for general SDF models

File: ur_handeye_simulation/urdf/ur_handeye_workcell.urdf.xacro (robot description, xacro)
@@ -78,4 +78,12 @@
     </xacro:handeye_pattern>
   </xacro:if>
+  <xacro:if value="${setup == 'none'}">
+    <xacro:handeye_camera
+      name="eye_in_hand_camera"
+      parent="tool0"
+    >
+      <origin xyz="0 -0.05 0.02" rpy="${pi/2} ${-pi/2} 0" />
+    </xacro:handeye_camera>
+  </xacro:if>
   <!-- ============================================================================ -->
   <!-- GAZEBO -->
